Commit message: made teleop node

File: src/ackermann_simulation/urdf/ackermann_car.urdf.xacro (robot description, xacro)
@@ -2,10 +2,10 @@
 <robot xmlns:xacro="http://ros.org/wiki/xacro" name="ackermann_robot">
   <!-- Include common macros (optional) -->
-  <xacro:property name="wheel_radius" value="0.1"/>
-  <xacro:property name="wheel_width" value="0.05"/>
+  <xacro:property name="wheel_radius" value="0.15"/>
+  <xacro:property name="wheel_width" value="0.1"/>
   <xacro:property name="chassis_length" value="1.0"/>
-  <xacro:property name="chassis_width" value="0.6"/>
+  <xacro:property name="chassis_width" value="0.4"/>
   <xacro:property name="chassis_height" value="0.15"/>
-  <xacro:property name="steering_link_length" value="0.2"/>
+  <xacro:property name="steering_link_length" value="0.6"/>
   <!-- Base Link -->
   <link name="base_link">
